Commit message: update v1.0

File: urdf/urdf.urdf (robot description, URDF)
Before this commit: robot urdf, 8 links, 7 joints
Links:
- removed link lindar
- added link base_footprint
- added link lidar, mass 0.146695752131392; collision mesh filename=package://final/meshes/lidar.STL; visual mesh filename=package://final/meshes/lidar.STL
- link Left_backward_wheel: geometry collision mesh filename=package://final/meshes/Left_backward_wheel.STL; visual mesh filename=package://final/meshes/Left_backward_wheel.STL
- link Left_forward_wheel: geometry collision mesh filename=package://final/meshes/Left_forward_wheel.STL; visual mesh filename=package://final/meshes/Left_forward_wheel.STL
- link Right_backward_wheel: geometry collision mesh filename=package://final/meshes/Right_backward_wheel.STL; visual mesh filename=package://final/meshes/Right_backward_wheel.STL
- link Right_forward_wheel: geometry collision mesh filename=package://final/meshes/Right_forward_wheel.STL; visual mesh filename=package://final/meshes/Right_forward_wheel.STL
- link base_link: geometry collision mesh filename=package://final/meshes/base_link.STL; visual mesh filename=package://final/meshes/base_link.STL
Joints:
- added joint base_footprint_to_base_link: type fixed, parent base_footprint, child base_link
- joint lidar_joint: child lindar -> lidar
